Commit message: Update ROS2 drone GNSS/INS simulation workspace

File: src/my_robot_description/urdf/my_robot.urdf.xacro (robot description, xacro)
@@ -6,4 +6,22 @@
     <xacro:property name="wheel_radius" value="0.1" />
     <xacro:property name="wheel_length" value="0.05" />
+    <xacro:macro name="box_inertia" params="m x y z o_xyz o_rpy">
+        <inertial>
+            <mass value="${m}" />
+            <origin xyz="${o_xyz}" rpy="${o_rpy}" />
+            <inertia ixx="${(m/12.0) * (y*y + z*z)}" ixy="0" ixz="0"
+                     iyy="${(m/12.0) * (x*x + z*z)}" iyz="0"
+                     izz="${(m/12.0) * (x*x + y*y)}" />
+        </inertial>
+    </xacro:macro>
+    <xacro:macro name="cylinder_inertia" params="m r h o_xyz o_rpy">
+        <inertial>
+            <mass value="${m}" />
+            <origin xyz="${o_xyz}" rpy="${o_rpy}" />
+            <inertia ixx="${(m/12.0) * (3*r*r + h*h)}" ixy="0" ixz="0"
+                     iyy="${(m/12.0) * (3*r*r + h*h)}" iyz="0"
+                     izz="${(m/2.0) * r*r}" />
+        </inertial>
+    </xacro:macro>
     <material name="green">
         <color rgba="0 0.5 0 1" />
@@ -21,9 +39,16 @@
             <material name="green" />
         </visual>
+        <collision>
+            <geometry>
+                <box size="${base_length} ${base_width} ${base_height}" />
+            </geometry>
+            <origin xyz="0.0 0.0 ${base_height / 2.0}" rpy="0 0 0" />
+        </collision>
+        <xacro:box_inertia m="5" x="${base_length}" y="${base_width}" z="${base_height}" o_xyz="0 0 ${base_height / 2.0}" o_rpy="0 0 0" />
     </link>
     <joint name="base_footprint_joint" type="fixed">
         <parent link="base_footprint" />
         <child link="base_link" />
-        <origin xyz="0 0 ${base_height / 2.0}" rpy="0 0 0" />
+        <origin xyz="0 0 ${wheel_radius}" rpy="0 0 0" />
     </joint>
     <xacro:macro name="wheel" params="prefix x_reflect y_reflect">
@@ -36,9 +61,16 @@
                 <material name="blue" />
             </visual>
+            <collision>
+                <geometry>
+                    <cylinder radius="${wheel_radius}" length="${wheel_length}" />
+                </geometry>
+                <origin xyz="0.0 0.0 0" rpy="1.5708 0 0" />
+            </collision>
+            <xacro:cylinder_inertia m="1" r="${wheel_radius}" h="${wheel_length}" o_xyz="0 0 0" o_rpy="1.5708 0 0" />
         </link>
         <joint name="base_${prefix}_wheel_joint" type="continuous">
             <parent link="base_link" />
             <child link="${prefix}_wheel_link" />
-            <origin xyz="${x_reflect * (base_length / 4.0)} ${y_reflect * 0.225} -${base_height / 2.0}" rpy="0 0 0" />
+            <origin xyz="${x_reflect * (base_length / 4.0)} ${y_reflect * 0.225} 0" rpy="0 0 0" />
             <axis xyz="0 1 0" />
         </joint>
@@ -48,3 +80,24 @@
     <xacro:wheel prefix="rear_right"  x_reflect="-1" y_reflect="-1" />
     <xacro:wheel prefix="rear_left"   x_reflect="-1" y_reflect="1" />
+    <gazebo>
+        <plugin name="gz::sim::systems::DiffDrive" filename="gz-sim-diff-drive-system">
+            <left_joint>base_front_left_wheel_joint</left_joint>
+            <left_joint>base_rear_left_wheel_joint</left_joint>
+            <right_joint>base_front_right_wheel_joint</right_joint>
+            <right_joint>base_rear_right_wheel_joint</right_joint>
+            <wheel_separation>0.45</wheel_separation>
+            <wheel_radius>0.1</wheel_radius>
+            <frame_id>odom</frame_id>
+            <child_frame_id>base_footprint</child_frame_id>
+            <topic>/model/my_robot/cmd_vel</topic>
+        </plugin>
+    </gazebo>
+    <gazebo>
+        <plugin name="gz::sim::systems::JointStatePublisher" filename="gz-sim-joint-state-publisher-system">
+            <joint_name>base_front_left_wheel_joint</joint_name>
+            <joint_name>base_front_right_wheel_joint</joint_name>
+            <joint_name>base_rear_left_wheel_joint</joint_name>
+            <joint_name>base_rear_right_wheel_joint</joint_name>
+        </plugin>
+    </gazebo>
 </robot>
