Commit message: Add diff_drive ros2_control, IMU, EKF sensor fusion, path visualization
- Replace DiffDrive Gazebo plugin with gz_ros2_control + ros2_control hardware interfaces
- Add IMU sensor (budget MEMS noise) to URDF
- Add gz::sim::systems::OdometryPublisher for ground truth pose
- Add EKF (robot_localization) fusing wheel odometry + IMU
- Add ekf_imu_only.yaml for comparison node
- Add gazebo_bridge.yaml: IMU + ground_truth/odom bridges
- Add ros2_control controllers config (diff_drive_controller, joint_state_broadcaster)
- Switch launch from XML to Python to avoid YAML-escaping issues with xacro
- Add square_move.py: closed-loop 2m x 2m square using EKF feedback
- Add odom_to_path.py: converts odometry topics to nav_msgs/Path for RViz
- Add imu_dead_reckoning.py: IMU heading dead-reckoning for comparison
- Update RViz config: Path displays for ground truth / wheel odom / EKF fused
- Fix IMU noise: budget MEMS level for visible sensor deviation

File: src/my_robot_description/urdf/my_robot.urdf.xacro (robot description, xacro)
@@ -1,4 +1,5 @@
 <?xml version="1.0"?>
 <robot name="my_robot" xmlns:xacro="http://www.ros.org/wiki/xacro">
+    <xacro:arg name="controllers_config" default="" />
     <xacro:property name="base_length" value="0.6" />
     <xacro:property name="base_width" value="0.4" />
@@ -83,23 +84,48 @@
     <xacro:wheel prefix="rear_right"  x_reflect="-1" y_reflect="-1" />
     <xacro:wheel prefix="rear_left"   x_reflect="-1" y_reflect="1" />
+    <!-- ==========================================
+         ros2_control hardware interfaces
+    ========================================== -->
+    <ros2_control name="GazeboSystem" type="system">
+        <hardware>
+            <plugin>gz_ros2_control/GazeboSimSystem</plugin>
+        </hardware>
+        <joint name="base_front_left_wheel_joint">
+            <command_interface name="velocity"/>
+            <state_interface name="position"/>
+            <state_interface name="velocity"/>
+        </joint>
+        <joint name="base_front_right_wheel_joint">
+            <command_interface name="velocity"/>
+            <state_interface name="position"/>
+            <state_interface name="velocity"/>
+        </joint>
+        <joint name="base_rear_left_wheel_joint">
+            <command_interface name="velocity"/>
+            <state_interface name="position"/>
+            <state_interface name="velocity"/>
+        </joint>
+        <joint name="base_rear_right_wheel_joint">
+            <command_interface name="velocity"/>
+            <state_interface name="position"/>
+            <state_interface name="velocity"/>
+        </joint>
+    </ros2_control>
+    <!-- gz_ros2_control plugin (starts controller_manager inside Gazebo) -->
     <gazebo>
-        <plugin name="gz::sim::systems::DiffDrive" filename="gz-sim-diff-drive-system">
-            <left_joint>base_front_left_wheel_joint</left_joint>
-            <left_joint>base_rear_left_wheel_joint</left_joint>
-            <right_joint>base_front_right_wheel_joint</right_joint>
-            <right_joint>base_rear_right_wheel_joint</right_joint>
-            <wheel_separation>0.45</wheel_separation>
-            <wheel_radius>0.1</wheel_radius>
-            <frame_id>odom</frame_id>
-            <child_frame_id>base_footprint</child_frame_id>
-            <topic>/model/my_robot/cmd_vel</topic>
+        <plugin filename="gz_ros2_control-system"
+                name="gz_ros2_control::GazeboSimROS2ControlPlugin">
+            <parameters>$(arg controllers_config)</parameters>
         </plugin>
     </gazebo>
+    <!-- Ground truth odometry from Gazebo model pose -->
     <gazebo>
-        <plugin name="gz::sim::systems::JointStatePublisher" filename="gz-sim-joint-state-publisher-system">
-            <joint_name>base_front_left_wheel_joint</joint_name>
-            <joint_name>base_front_right_wheel_joint</joint_name>
-            <joint_name>base_rear_left_wheel_joint</joint_name>
-            <joint_name>base_rear_right_wheel_joint</joint_name>
+        <plugin filename="gz-sim-odometry-publisher-system"
+                name="gz::sim::systems::OdometryPublisher">
+            <odom_frame>odom</odom_frame>
+            <robot_base_frame>base_footprint</robot_base_frame>
+            <odom_topic>/model/my_robot/ground_truth/odom</odom_topic>
+            <tf_topic>/model/my_robot/ground_truth/tf</tf_topic>
+            <odom_publish_frequency>50</odom_publish_frequency>
         </plugin>
     </gazebo>
@@ -210,3 +236,66 @@
         </sensor>
     </gazebo>
+    <!-- ==========================================
+         IMU SENSOR
+    ========================================== -->
+    <link name="imu_link">
+        <visual>
+            <geometry>
+                <box size="0.05 0.05 0.02" />
+            </geometry>
+            <material name="red" />
+        </visual>
+        <collision>
+            <geometry>
+                <box size="0.05 0.05 0.02" />
+            </geometry>
+        </collision>
+        <xacro:box_inertia m="0.05" x="0.05" y="0.05" z="0.02"
+                           o_xyz="0 0 0" o_rpy="0 0 0" />
+    </link>
+    <joint name="base_imu_joint" type="fixed">
+        <parent link="base_link" />
+        <child link="imu_link" />
+        <origin xyz="0 0 ${base_height}" rpy="0 0 0" />
+    </joint>
+    <gazebo reference="imu_link">
+        <sensor name="imu_sensor" type="imu">
+            <always_on>1</always_on>
+            <update_rate>100</update_rate>
+            <visualize>false</visualize>
+            <topic>imu</topic>
+            <gz_frame_id>imu_link</gz_frame_id>
+            <imu>
+                <!-- Noise: budget consumer MEMS level - produces visible deviation -->
+                <angular_velocity>
+                    <x><noise type="gaussian">
+                        <mean>0.0</mean><stddev>0.009</stddev>
+                        <bias_mean>0.03</bias_mean><bias_stddev>0.005</bias_stddev>
+                    </noise></x>
+                    <y><noise type="gaussian">
+                        <mean>0.0</mean><stddev>0.009</stddev>
+                        <bias_mean>0.03</bias_mean><bias_stddev>0.005</bias_stddev>
+                    </noise></y>
+                    <z><noise type="gaussian">
+                        <mean>0.0</mean><stddev>0.009</stddev>
+                        <bias_mean>0.03</bias_mean><bias_stddev>0.005</bias_stddev>
+                    </noise></z>
+                </angular_velocity>
+                <linear_acceleration>
+                    <x><noise type="gaussian">
+                        <mean>0.0</mean><stddev>0.065</stddev>
+                        <bias_mean>0.18</bias_mean><bias_stddev>0.015</bias_stddev>
+                    </noise></x>
+                    <y><noise type="gaussian">
+                        <mean>0.0</mean><stddev>0.065</stddev>
+                        <bias_mean>0.18</bias_mean><bias_stddev>0.015</bias_stddev>
+                    </noise></y>
+                    <z><noise type="gaussian">
+                        <mean>0.0</mean><stddev>0.065</stddev>
+                        <bias_mean>0.18</bias_mean><bias_stddev>0.015</bias_stddev>
+                    </noise></z>
+                </linear_acceleration>
+            </imu>
+        </sensor>
+    </gazebo>
 </robot>
